File: USB-C-Android-head-unit/power.sch (KiCad schematic (older format))
At the start: 0 parts

Commit message: starting usb c design
Other:
- note added: "VBUS is power input from one and only one USB C jack at a time."
Changed lines of the file:
@@
 EESchema Schematic File Version 4
+LIBS:USB-C-Android-head-unit-cache
 EELAYER 30 0
 EELAYER END
 $Descr A4 11693 8268
 encoding utf-8
-Sheet 1 5
+Sheet 4 7
 Title ""
 Date ""
@@
 Comment4 ""
 $EndDescr
+$Comp
+L power:VBUS #PWR?
+U 1 1 5D79D030
+P 6850 2750
+F 0 "#PWR?" H 6850 2600 50  0001 C CNN
+F 1 "VBUS" H 6850 2900 50  0000 C CNN
+F 2 "" H 6850 2750 50  0001 C CNN
+F 3 "" H 6850 2750 50  0001 C CNN
+	1    6850 2750
+	1    0    0    -1
+$EndComp
+Text Notes 4550 3450 0    50   ~ 0
+VBUS is power input from one and only one USB C jack at a time.
 $EndSCHEMATC
